Commit message: work_29_09_2021

File: mrcp_trex_gripper/mrcp_trex_gripper_description/urdf/mrcp_trex_gripper.urdf (robot description, URDF)
Before this commit: robot roverv1, 15 links, 14 joints
Links:
- added link body_footprint
- added link link_1, mass 2.9455; collision mesh filename=package://mrcp_trex_gripper_description/meshes/link_1.STL scale=1 1 1; visual mesh filename=package://mrcp_trex_gripper_description/meshes/link_1.STL scale=1 1 1
- added link link_2, mass 2.9623; collision mesh filename=package://mrcp_trex_gripper_description/meshes/link_2.STL scale=1 1 1; visual mesh filename=package://mrcp_trex_gripper_description/meshes/link_2.STL scale=1 1 1
- added link link_3, mass 2.0676; collision mesh filename=package://mrcp_trex_gripper_description/meshes/link_3.STL scale=1 1 1; visual mesh filename=package://mrcp_trex_gripper_description/meshes/link_3.STL scale=1 1 1
- added link link_4, mass 0.9251; collision mesh filename=package://mrcp_trex_gripper_description/meshes/link_4.STL scale=1 1 1; visual mesh filename=package://mrcp_trex_gripper_description/meshes/link_4.STL scale=1 1 1
- added link link_5, mass 0.69913; collision mesh filename=package://mrcp_trex_gripper_description/meshes/link_5.STL scale=1 1 1; visual mesh filename=package://mrcp_trex_gripper_description/meshes/link_5.STL scale=1 1 1
- added link link_6, mass 0.30019; collision mesh filename=package://mrcp_trex_gripper_description/meshes/link_6.STL scale=1 1 1; visual mesh filename=package://mrcp_trex_gripper_description/meshes/link_6.STL scale=1 1 1
- link Left_Bogie: geometry collision mesh filename=package://mrcp_trex_gripper_description/meshes/RSArm.STL scale=1 1 1; visual mesh filename=package://mrcp_trex_gripper_description/meshes/RSArm.STL scale=1 1 1
- link Left_Rocker: geometry collision mesh filename=package://mrcp_trex_gripper_description/meshes/RLArm.STL scale=1 1 1; visual mesh filename=package://mrcp_trex_gripper_description/meshes/RLArm.STL scale=1 1 1
- link Right_Bogie: geometry collision mesh filename=package://mrcp_trex_gripper_description/meshes/LSArm.STL scale=1 1 1; visual mesh filename=package://mrcp_trex_gripper_description/meshes/LSArm.STL scale=1 1 1
- link Right_Rocker: geometry collision mesh filename=package://mrcp_trex_gripper_description/meshes/LLArm.STL scale=1 1 1; visual mesh filename=package://mrcp_trex_gripper_description/meshes/LLArm.STL scale=1 1 1
- link Servo1: geometry collision mesh filename=package://mrcp_trex_gripper_description/meshes/StWh1.STL scale=1 1 1; visual mesh filename=package://mrcp_trex_gripper_description/meshes/StWh1.STL scale=1 1 1
- link Servo2: geometry collision mesh filename=package://mrcp_trex_gripper_description/meshes/StWh1.STL scale=1 1 1; visual mesh filename=package://mrcp_trex_gripper_description/meshes/StWh1.STL scale=1 1 1
- link Servo3: geometry collision mesh filename=package://mrcp_trex_gripper_description/meshes/StWh1.STL scale=1 1 1; visual mesh filename=package://mrcp_trex_gripper_description/meshes/StWh1.STL scale=1 1 1
- link Servo4: geometry collision mesh filename=package://mrcp_trex_gripper_description/meshes/StWh1.STL scale=1 1 1; visual mesh filename=package://mrcp_trex_gripper_description/meshes/StWh1.STL scale=1 1 1
- link Wheel1: geometry collision mesh filename=package://mrcp_trex_gripper_description/meshes/Wheel.STL scale=1 1 1; visual mesh filename=package://mrcp_trex_gripper_description/meshes/Wheel.STL scale=1 1 1
- link Wheel2: geometry collision mesh filename=package://mrcp_trex_gripper_description/meshes/Wheel.STL scale=1 1 1; visual mesh filename=package://mrcp_trex_gripper_description/meshes/Wheel.STL scale=1 1 1
- link Wheel3: geometry collision mesh filename=package://mrcp_trex_gripper_description/meshes/Wheel.STL scale=1 1 1; visual mesh filename=package://mrcp_trex_gripper_description/meshes/Wheel.STL scale=1 1 1
- link Wheel4: geometry collision mesh filename=package://mrcp_trex_gripper_description/meshes/Wheel.STL scale=1 1 1; visual mesh filename=package://mrcp_trex_gripper_description/meshes/Wheel.STL scale=1 1 1
- link Wheel5: geometry collision mesh filename=package://mrcp_trex_gripper_description/meshes/Wheel.STL scale=1 1 1; visual mesh filename=package://mrcp_trex_gripper_description/meshes/Wheel.STL scale=1 1 1
- link Wheel6: geometry collision mesh filename=package://mrcp_trex_gripper_description/meshes/Wheel.STL scale=1 1 1; visual mesh filename=package://mrcp_trex_gripper_description/meshes/Wheel.STL scale=1 1 1
- link body: geometry collision mesh filename=package://mrcp_trex_gripper_description/meshes/base.STL scale=1 1 1; visual mesh filename=package://mrcp_trex_gripper_description/meshes/base.STL scale=1 1 1
Joints:
- added joint arm_base_joint: type fixed, parent body, child link_1, origin xyz=0 0 0.25 rpy=0 0 0
- added joint fixed: type fixed, parent body_footprint, child body, origin xyz=0 0 0.3 rpy=0 0 0
- added joint joint_1: type revolute, parent link_1, child link_2, origin xyz=-0.0085035 0.003 0.072 rpy=0 0 0, axis 0 0 -1, limit lower=-3.14 upper=3.14 effort=87 velocity=2.1750
- added joint joint_2: type revolute, parent link_2, child link_3, origin xyz=0.0043365 -0.033328 0.0579 rpy=0 0 0, axis 0.12903 -0.99164 0, limit lower=-0.47 upper=1.57 effort=87 velocity=2.1750
- added joint joint_3: type revolute, parent link_3, child link_4, origin xyz=0.1495 0.050117 0.25703 rpy=0 0 0, axis 0.12903 -0.99164 0, limit lower=-0.9 upper=1.5 effort=87 velocity=2.1750
- added joint joint_4: type revolute, parent link_4, child link_5, origin xyz=0.22469 0.0072929 0.023651 rpy=0 0 0, axis 0.12903 -0.99164 0, limit lower=-0.9 upper=3.14 effort=87 velocity=2.1750
- added joint joint_5: type revolute, parent link_5, child link_6, origin xyz=0.041015 0.029287 -0.094022 rpy=0 0 0, axis 0.42384 0.05515 -0.90406, limit lower=-3.14 upper=3.14 effort=87 velocity=2.1750
- joint Left_Rocker_joint: type revolute -> fixed
- joint Right_Rocker_joint: type revolute -> fixed

File: trex_gripper/roverv1/urdf/mrcp_trex_moving.urdf (robot description, URDF)
Before this commit: robot roverv1, 16 links, 15 joints
Links:
- added link link_1, mass 2.9455; collision mesh filename=package://mrcp_trex_gripper_description/meshes/link_1.STL scale=1 1 1; visual mesh filename=package://mrcp_trex_gripper_description/meshes/link_1.STL scale=1 1 1
- added link link_2, mass 2.9623; collision mesh filename=package://mrcp_trex_gripper_description/meshes/link_2.STL scale=1 1 1; visual mesh filename=package://mrcp_trex_gripper_description/meshes/link_2.STL scale=1 1 1
- added link link_3, mass 2.0676; collision mesh filename=package://mrcp_trex_gripper_description/meshes/link_3.STL scale=1 1 1; visual mesh filename=package://mrcp_trex_gripper_description/meshes/link_3.STL scale=1 1 1
- added link link_4, mass 0.9251; collision mesh filename=package://mrcp_trex_gripper_description/meshes/link_4.STL scale=1 1 1; visual mesh filename=package://mrcp_trex_gripper_description/meshes/link_4.STL scale=1 1 1
- added link link_5, mass 0.69913; collision mesh filename=package://mrcp_trex_gripper_description/meshes/link_5.STL scale=1 1 1; visual mesh filename=package://mrcp_trex_gripper_description/meshes/link_5.STL scale=1 1 1
- added link link_6, mass 0.30019; collision mesh filename=package://mrcp_trex_gripper_description/meshes/link_6.STL scale=1 1 1; visual mesh filename=package://mrcp_trex_gripper_description/meshes/link_6.STL scale=1 1 1
Joints:
- added joint arm_base_joint: type fixed, parent body, child link_1, origin xyz=0 0 0.25 rpy=0 0 0
- added joint joint_1: type revolute, parent link_1, child link_2, origin xyz=-0.0085035 0.003 0.072 rpy=0 0 0, axis 0 0 -1, limit lower=-3.14 upper=3.14 effort=87 velocity=2.1750
- added joint joint_2: type revolute, parent link_2, child link_3, origin xyz=0.0043365 -0.033328 0.0579 rpy=0 0 0, axis 0.12903 -0.99164 0, limit lower=-0.47 upper=1.57 effort=87 velocity=2.1750
- added joint joint_3: type revolute, parent link_3, child link_4, origin xyz=0.1495 0.050117 0.25703 rpy=0 0 0, axis 0.12903 -0.99164 0, limit lower=-0.9 upper=1.5 effort=87 velocity=2.1750
- added joint joint_4: type revolute, parent link_4, child link_5, origin xyz=0.22469 0.0072929 0.023651 rpy=0 0 0, axis 0.12903 -0.99164 0, limit lower=-0.9 upper=3.14 effort=87 velocity=2.1750
- added joint joint_5: type revolute, parent link_5, child link_6, origin xyz=0.041015 0.029287 -0.094022 rpy=0 0 0, axis 0.42384 0.05515 -0.90406, limit lower=-3.14 upper=3.14 effort=87 velocity=2.1750
